File: tailboard_signalling_pcb/tailboard_signalling_pcb.sch (KiCad schematic (older format))
At the start: 22 parts, among them J1 Conn_Coaxial, J2 Conn_Coaxial_Power, U1 SN75176AD, U2 LDO_ILC7080, X1 RJ45, X2 USB_A, Y1 XRCGB24M000F0L00R0

Commit message: del
Parts:
- D1, U2: footprint signal_EE285:SOT23-5 -> tailboard_signalling_pcb:SOT23-5
- D2: footprint signal_EE285:SOP-14 -> tailboard_signalling_pcb:SOP-14
Changed lines of the file:
@@
 F 0 "D1" H 8900 2615 50  0000 C CNN
 F 1 "IRU1205-33" H 8900 2524 50  0000 C CNN
-F 2 "signal_EE285:SOT23-5" H 8900 2550 50  0001 C CNN
+F 2 "tailboard_signalling_pcb:SOT23-5" H 8900 2550 50  0001 C CNN
 F 3 "" H 8900 1950 50  0001 C CNN
 	1    8900 2250
@@
 F 0 "D2" H 7350 4600 50  0000 C CNN
 F 1 "UIC4102CP" H 7350 4500 50  0000 C CNN
-F 2 "signal_EE285:SOP-14" H 7350 4650 50  0001 C CNN
+F 2 "tailboard_signalling_pcb:SOP-14" H 7350 4650 50  0001 C CNN
 F 3 "" H 7350 4550 50  0001 C CNN
 	1    7350 4050
@@
 F 0 "U2" H 2250 6900 50  0000 L CNN
 F 1 "LDO_ILC7080" H 2050 6750 50  0000 L CNN
-F 2 "signal_EE285:SOT23-5" H 2300 6600 50  0001 C CNN
+F 2 "tailboard_signalling_pcb:SOT23-5" H 2300 6600 50  0001 C CNN
 F 3 "" H 2300 6600 50  0001 C CNN
 	1    2300 6350
